Commit message: update

File: tianyi2_urdf/urdf/tianyi2.0_URDF.urdf (robot description, URDF)
Before this commit: robot tianyi2_urdf, 25 links, 24 joints
Links:
- removed link body_yaw_link
- added link waist_yaw_link, mass 13.795395; collision mesh filename=package://tianyi2_urdf/meshes_convex/waist_yaw_link.STL; visual mesh filename=package://tianyi2_urdf/meshes/waist_yaw_link.STL
- link base: geometry collision mesh filename=package://tianyi2_urdf/meshes_convex/base.STL; visual mesh filename=package://tianyi2_urdf/meshes/base.STL
- link camera_head_link: geometry collision mesh filename=package://tianyi2_urdf/meshes_convex/camera_head_link.STL; visual mesh filename=package://tianyi2_urdf/meshes/camera_head_link.STL
- link elbow_pitch_l_link: geometry collision mesh filename=package://tianyi2_urdf/meshes_convex/elbow_pitch_l_link.STL; visual mesh filename=package://tianyi2_urdf/meshes/elbow_pitch_l_link.STL
- link elbow_pitch_r_link: geometry collision mesh filename=package://tianyi2_urdf/meshes_convex/elbow_pitch_r_link.STL; visual mesh filename=package://tianyi2_urdf/meshes/elbow_pitch_r_link.STL
- link elbow_yaw_l_link: geometry collision mesh filename=package://tianyi2_urdf/meshes_convex/elbow_yaw_l_link.STL; visual mesh filename=package://tianyi2_urdf/meshes/elbow_yaw_l_link.STL
- link elbow_yaw_r_link: geometry collision mesh filename=package://tianyi2_urdf/meshes_convex/elbow_yaw_r_link.STL; visual mesh filename=package://tianyi2_urdf/meshes/elbow_yaw_r_link.STL
- link first_leg_pitch_link: geometry collision mesh filename=package://tianyi2_urdf/meshes_convex/first_leg_pitch_link.S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; visual mesh filename=package://tianyi2_urdf/meshes/first_leg_pitch_link.STL
- link head_pitch_link: geometry collision mesh filename=package://tianyi2_urdf/meshes_convex/head_pitch_link.STL; visual mesh filename=package://tianyi2_urdf/meshes/head_pitch_link.STL
- link head_roll_link: geometry collision mesh filename=package://tianyi2_urdf/meshes_convex/head_roll_link.STL; visual mesh filename=package://tianyi2_urdf/meshes/head_roll_link.STL
- link head_yaw_link: geometry collision mesh filename=package://tianyi2_urdf/meshes_convex/head_yaw_link.STL; visual mesh filename=package://tianyi2_urdf/meshes/head_yaw_link.STL
- link left_tcp_link: geometry collision mesh filename=package://tianyi2_urdf/meshes_convex/left_tcp_link.STL; visual mesh filename=package://tianyi2_urdf/meshes/left_tcp_link.STL
- link right_tcp_link: geometry collision mesh filename=package://tianyi2_urdf/meshes_convex/right_tcp_link.STL; visual mesh filename=package://tianyi2_urdf/meshes/right_tcp_link.STL
- link second_leg_pitch_link: geometry collision mesh filename=package://tianyi2_urdf/meshes_convex/second_leg_pitch_link.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; visual mesh filename=package://tianyi2_urdf/meshes/second_leg_pitch_link.STL
- link shoulder_pitch_l_link: geometry collision mesh filename=package://tianyi2_urdf/meshes_convex/shoulder_pitch_l_link.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; visual mesh filename=package://tianyi2_urdf/meshes/shoulder_pitch_l_link.STL
- link shoulder_pitch_r_link: geometry collision mesh filename=package://tianyi2_urdf/meshes_convex/shoulder_pitch_r_link.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; visual mesh filename=package://tianyi2_urdf/meshes/shoulder_pitch_r_link.STL
- link shoulder_roll_l_link: geometry collision mesh filename=package://tianyi2_urdf/meshes_convex/shoulder_roll_l_link.S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; visual mesh filename=package://tianyi2_urdf/meshes/shoulder_roll_l_link.STL
- link shoulder_roll_r_link: geometry collision mesh filename=package://tianyi2_urdf/meshes_convex/shoulder_roll_r_link.S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; visual mesh filename=package://tianyi2_urdf/meshes/shoulder_roll_r_link.STL
- link shoulder_yaw_l_link: geometry collision mesh filename=package://tianyi2_urdf/meshes_convex/shoulder_yaw_l_link.STL; visual mesh filename=package://tianyi2_urdf/meshes/shoulder_yaw_l_link.STL
- link shoulder_yaw_r_link: geometry collision mesh filename=package://tianyi2_urdf/meshes_convex/shoulder_yaw_r_link.STL; visual mesh filename=package://tianyi2_urdf/meshes/shoulder_yaw_r_link.STL
- link waist_pitch_link: geometry collision mesh filename=package://tianyi2_urdf/meshes_convex/waist_pitch_link.STL; visual mesh filename=package://tianyi2_urdf/meshes/waist_pitch_link.STL
- link wrist_pitch_l_link: geometry collision mesh filename=package://tianyi2_urdf/meshes_convex/wrist_pitch_l_link.STL; visual mesh filename=package://tianyi2_urdf/meshes/wrist_pitch_l_link.STL
- link wrist_pitch_r_link: geometry collision mesh filename=package://tianyi2_urdf/meshes_convex/wrist_pitch_r_link.STL; visual mesh filename=package://tianyi2_urdf/meshes/wrist_pitch_r_link.STL
- link wrist_roll_l_link: geometry collision mesh filename=package://tianyi2_urdf/meshes_convex/wrist_roll_l_link.STL; visual mesh filename=package://tianyi2_urdf/meshes/wrist_roll_l_link.STL
- link wrist_roll_r_link: geometry collision mesh filename=package://tianyi2_urdf/meshes_convex/wrist_roll_r_link.STL; visual mesh filename=package://tianyi2_urdf/meshes/wrist_roll_r_link.STL
Joints:
- removed joint body_yaw_joint
- added joint waist_yaw_joint: type revolute, parent waist_pitch_link, child waist_yaw_link, origin xyz=0 0 0.07 rpy=0 0 0, axis 0 0 1, limit lower=-2.9670597283903604 upper=3.141592653589793 effort=143.0 velocity=4.71238898038469
- joint first_leg_pitch_joint: limit lower=-0.41887902047863906 upper=1.0471975511965976 effort=332.0 velocity=3.9269908169872414 -> lower=-0.41887902047863906 upper=0.9075712110370514 effort=332.0 velocity=3.9269908169872414
- joint head_yaw_joint: parent body_yaw_link -> waist_yaw_link
- joint second_leg_pitch_joint: limit lower=-0.5061454830783556 upper=1.7453292519943295 effort=332.0 velocity=3.9269908169872414 -> lower=-1.7453292519943295 upper=0.5061454830783556 effort=332.0 velocity=3.9269908169872414
- joint shoulder_pitch_l_joint: parent body_yaw_link -> waist_yaw_link
- joint shoulder_pitch_r_joint: parent body_yaw_link -> waist_yaw_link
- joint shoulder_roll_l_joint: limit lower=-1.0471975511965976 upper=1.8325957145940461 effort=95.0 velocity=3.979350694547071 -> lower=-0.2617993877991494 upper=2.6179938779914944 effort=95.0 velocity=3.979350694547071
- joint shoulder_roll_r_joint: limit lower=-1.8325957145940461 upper=1.0471975511965976 effort=95.0 velocity=3.979350694547071 -> lower=-2.6179938779914944 upper=0.2617993877991494 effort=95.0 velocity=3.979350694547071
- joint waist_pitch_joint: limit lower=-2.0943951023931953 upper=0.7853981633974483 effort=332.0 velocity=3.9269908169872414 -> lower=-0.7853981633974483 upper=2.0943951023931953 effort=332.0 velocity=3.9269908169872414
- joint wrist_pitch_l_joint: limit lower=-1.3089969389957472 upper=1.6580627893946132 effort=6.3 velocity=7.5398223686155035 -> lower=-0.7853981633974483 upper=1.0471975511965976 effort=6.3 velocity=7.5398223686155035
- joint wrist_pitch_r_joint: limit lower=-1.3089969389957472 upper=1.6580627893946132 effort=6.3 velocity=7.5398223686155035 -> lower=-0.7853981633974483 upper=1.0471975511965976 effort=6.3 velocity=7.5398223686155035
- joint wrist_roll_l_joint: limit lower=-1.0471975511965976 upper=0.7853981633974483 effort=6.3 velocity=7.5398223686155035 -> lower=-1.6580627893946132 upper=1.3089969389957472 effort=6.3 velocity=7.5398223686155035
- joint wrist_roll_r_joint: limit lower=-0.7853981633974483 upper=1.0471975511965976 effort=6.3 velocity=7.5398223686155035 -> lower=-1.3089969389957472 upper=1.6580627893946132 effort=6.3 velocity=7.5398223686155035

File: tianyi2_urdf/urdf/tianyi2.0_URDF.urdf.xacro (robot description, xacro)
@@ -19,5 +19,5 @@
       <origin xyz="0 0 0" rpy="0 0 0" />
       <geometry>
-        <mesh filename="package://tianyi2_urdf/meshes/base.STL" />
+        <mesh filename="package://tianyi2_urdf/meshes_convex/base.STL" />
       </geometry>
     </collision>
@@ -41,5 +41,5 @@
       <origin xyz="0 0 0" rpy="0 0 0" />
       <geometry>
-        <mesh filename="package://tianyi2_urdf/meshes/first_leg_pitch_link.STL" />
+        <mesh filename="package://tianyi2_urdf/meshes_convex/first_leg_pitch_link.STL" />
       </geometry>
     </collision>
@@ -50,5 +50,5 @@
     <child link="first_leg_pitch_link" />
     <axis xyz="0 1 0" />
-    <limit lower="-0.41887902047863906" upper="1.0471975511965976" effort="332.0" velocity="3.9269908169872414" />
+    <limit lower="-0.41887902047863906" upper="0.9075712110370514" effort="332.0" velocity="3.9269908169872414" />
   </joint>
   <link name="second_leg_pitch_link">
@@ -70,5 +70,5 @@
       <origin xyz="0 0 0" rpy="0 0 0" />
       <geometry>
-        <mesh filename="package://tianyi2_urdf/meshes/second_leg_pitch_link.STL" />
+        <mesh filename="package://tianyi2_urdf/meshes_convex/second_leg_pitch_link.STL" />
       </geometry>
     </collision>
@@ -79,5 +79,5 @@
     <child link="second_leg_pitch_link" />
     <axis xyz="0 1 0" />
-    <limit lower="-0.5061454830783556" upper="1.7453292519943295" effort="332.0" velocity="3.9269908169872414" />
+    <limit lower="-1.7453292519943295" upper="0.5061454830783556" effort="332.0" velocity="3.9269908169872414" />
   </joint>
   <link name="waist_pitch_link">
@@ -99,5 +99,5 @@
       <origin xyz="0 0 0" rpy="0 0 0" />
       <geometry>
-        <mesh filename="package://tianyi2_urdf/meshes/waist_pitch_link.STL" />
+        <mesh filename="package://tianyi2_urdf/meshes_convex/waist_pitch_link.STL" />
       </geometry>
     </collision>
@@ -108,7 +108,7 @@
     <child link="waist_pitch_link" />
     <axis xyz="0 1 0" />
-    <limit lower="-2.0943951023931953" upper="0.7853981633974483" effort="332.0" velocity="3.9269908169872414" />
-  </joint>
-  <link name="body_yaw_link">
+    <limit lower="-0.7853981633974483" upper="2.0943951023931953" effort="332.0" velocity="3.9269908169872414" />
+  </joint>
+  <link name="waist_yaw_link">
     <inertial>
       <origin xyz="0.009196 -0.000592 0.251379" rpy="0 0 0" />
@@ -119,21 +119,21 @@
       <origin xyz="0 0 0" rpy="0 0 0" />
       <geometry>
-        <mesh filename="package://tianyi2_urdf/meshes/body_yaw_link.STL" />
-      </geometry>
-      <material name="">
-        <color rgba="0.752941176470588 0.752941176470588 0.752941176470588 1" />
-      </material>
-    </visual>
-    <collision>
-      <origin xyz="0 0 0" rpy="0 0 0" />
-      <geometry>
-        <mesh filename="package://tianyi2_urdf/meshes/body_yaw_link.STL" />
-      </geometry>
-    </collision>
-  </link>
-  <joint name="body_yaw_joint" type="revolute">
+        <mesh filename="package://tianyi2_urdf/meshes/waist_yaw_link.STL" />
+      </geometry>
+      <material name="">
+        <color rgba="0.752941176470588 0.752941176470588 0.752941176470588 1" />
+      </material>
+    </visual>
+    <collision>
+      <origin xyz="0 0 0" rpy="0 0 0" />
+      <geometry>
+        <mesh filename="package://tianyi2_urdf/meshes_convex/waist_yaw_link.STL" />
+      </geometry>
+    </collision>
+  </link>
+  <joint name="waist_yaw_joint" type="revolute">
     <origin xyz="0 0 0.07" rpy="0 0 0" />
     <parent link="waist_pitch_link" />
-    <child link="body_yaw_link" />
+    <child link="waist_yaw_link" />
     <axis xyz="0 0 1" />
     <limit lower="-2.9670597283903604" upper="3.141592653589793" effort="143.0" velocity="4.71238898038469" />
@@ -157,5 +157,5 @@
       <origin xyz="0 0 0" rpy="0 0 0" />
       <geometry>
-        <mesh filename="package://tianyi2_urdf/meshes/head_yaw_link.STL" />
+        <mesh filename="package://tianyi2_urdf/meshes_convex/head_yaw_link.STL" />
       </geometry>
     </collision>
@@ -163,5 +163,5 @@
   <joint name="head_yaw_joint" type="revolute">
     <origin xyz="-0.002 0 0.56508" rpy="0 0 0" />
-    <parent link="body_yaw_link" />
+    <parent link="waist_yaw_link" />
     <child link="head_yaw_link" />
     <axis xyz="0 0 1" />
@@ -186,5 +186,5 @@
       <origin xyz="0 0 0" rpy="0 0 0" />
       <geometry>
-        <mesh filename="package://tianyi2_urdf/meshes/head_pitch_link.STL" />
+        <mesh filename="package://tianyi2_urdf/meshes_convex/head_pitch_link.STL" />
       </geometry>
     </collision>
@@ -215,5 +215,5 @@
       <origin xyz="0 0 0" rpy="0 0 0" />
       <geometry>
-        <mesh filename="package://tianyi2_urdf/meshes/head_roll_link.STL" />
+        <mesh filename="package://tianyi2_urdf/meshes_convex/head_roll_link.STL" />
       </geometry>
     </collision>
@@ -244,5 +244,5 @@
       <origin xyz="0 0 0" rpy="0 0 0" />
       <geometry>
-        <mesh filename="package://tianyi2_urdf/meshes/camera_head_link.STL" />
+        <mesh filename="package://tianyi2_urdf/meshes_convex/camera_head_link.STL" />
       </geometry>
     </collision>
@@ -272,5 +272,5 @@
       <origin xyz="0 0 0" rpy="0 0 0" />
       <geometry>
-        <mesh filename="package://tianyi2_urdf/meshes/shoulder_pitch_l_link.STL" />
+        <mesh filename="package://tianyi2_urdf/meshes_convex/shoulder_pitch_l_link.STL" />
       </geometry>
     </collision>
@@ -278,5 +278,5 @@
   <joint name="shoulder_pitch_l_joint" type="revolute">
     <origin xyz="0 0.14539 0.37721" rpy="0.087266 0 0" />
-    <parent link="body_yaw_link" />
+    <parent link="waist_yaw_link" />
     <child link="shoulder_pitch_l_link" />
     <axis xyz="0 1 0" />
@@ -301,5 +301,5 @@
       <origin xyz="0 0 0" rpy="0 0 0" />
       <geometry>
-        <mesh filename="package://tianyi2_urdf/meshes/shoulder_roll_l_link.STL" />
+        <mesh filename="package://tianyi2_urdf/meshes_convex/shoulder_roll_l_link.STL" />
       </geometry>
     </collision>
@@ -310,5 +310,5 @@
     <child link="shoulder_roll_l_link" />
     <axis xyz="1 0 0" />
-    <limit lower="-1.0471975511965976" upper="1.8325957145940461" effort="95.0" velocity="3.979350694547071" />
+    <limit lower="-0.2617993877991494" upper="2.6179938779914944" effort="95.0" velocity="3.979350694547071" />
   </joint>
   <link name="shoulder_yaw_l_link">
@@ -330,5 +330,5 @@
       <origin xyz="0 0 0" rpy="0 0 0" />
       <geometry>
-        <mesh filename="package://tianyi2_urdf/meshes/shoulder_yaw_l_link.STL" />
+        <mesh filename="package://tianyi2_urdf/meshes_convex/shoulder_yaw_l_link.STL" />
       </geometry>
     </collision>
@@ -359,5 +359,5 @@
       <origin xyz="0 0 0" rpy="0 0 0" />
       <geometry>
-        <mesh filename="package://tianyi2_urdf/meshes/elbow_pitch_l_link.STL" />
+        <mesh filename="package://tianyi2_urdf/meshes_convex/elbow_pitch_l_link.STL" />
       </geometry>
     </collision>
@@ -388,5 +388,5 @@
       <origin xyz="0 0 0" rpy="0 0 0" />
       <geometry>
-        <mesh filename="package://tianyi2_urdf/meshes/elbow_yaw_l_link.STL" />
+        <mesh filename="package://tianyi2_urdf/meshes_convex/elbow_yaw_l_link.STL" />
       </geometry>
     </collision>
@@ -417,5 +417,5 @@
       <origin xyz="0 0 0" rpy="0 0 0" />
       <geometry>
-        <mesh filename="package://tianyi2_urdf/meshes/wrist_pitch_l_link.STL" />
+        <mesh filename="package://tianyi2_urdf/meshes_convex/wrist_pitch_l_link.STL" />
       </geometry>
     </collision>
@@ -426,5 +426,5 @@
     <child link="wrist_pitch_l_link" />
     <axis xyz="0 1 0" />
-    <limit lower="-1.3089969389957472" upper="1.6580627893946132" effort="6.3" velocity="7.5398223686155035" />
+    <limit lower="-0.7853981633974483" upper="1.0471975511965976" effort="6.3" velocity="7.5398223686155035" />
   </joint>
   <link name="wrist_roll_l_link">
@@ -446,5 +446,5 @@
       <origin xyz="0 0 0" rpy="0 0 0" />
       <geometry>
-        <mesh filename="package://tianyi2_urdf/meshes/wrist_roll_l_link.STL" />
+        <mesh filename="package://tianyi2_urdf/meshes_convex/wrist_roll_l_link.STL" />
       </geometry>
     </collision>
@@ -455,5 +455,5 @@
     <child link="wrist_roll_l_link" />
     <axis xyz="1 0 0" />
-    <limit lower="-1.0471975511965976" upper="0.7853981633974483" effort="6.3" velocity="7.5398223686155035" />
+    <limit lower="-1.6580627893946132" upper="1.3089969389957472" effort="6.3" velocity="7.5398223686155035" />
   </joint>
   <link name="left_tcp_link">
@@ -475,5 +475,5 @@
       <origin xyz="0 0 0" rpy="0 0 0" />
       <geometry>
-        <mesh filename="package://tianyi2_urdf/meshes/left_tcp_link.STL" />
+        <mesh filename="package://tianyi2_urdf/meshes_convex/left_tcp_link.STL" />
       </geometry>
     </collision>
@@ -503,5 +503,5 @@
       <origin xyz="0 0 0" rpy="0 0 0" />
       <geometry>
-        <mesh filename="package://tianyi2_urdf/meshes/shoulder_pitch_r_link.STL" />
+        <mesh filename="package://tianyi2_urdf/meshes_convex/shoulder_pitch_r_link.STL" />
       </geometry>
     </collision>
@@ -509,5 +509,5 @@
   <joint name="shoulder_pitch_r_joint" type="revolute">
     <origin xyz="0 -0.14539 0.37721" rpy="-0.087266 0 0" />
-    <parent link="body_yaw_link" />
+    <parent link="waist_yaw_link" />
     <child link="shoulder_pitch_r_link" />
     <axis xyz="0 1 0" />
@@ -532,5 +532,5 @@
       <origin xyz="0 0 0" rpy="0 0 0" />
       <geometry>
-        <mesh filename="package://tianyi2_urdf/meshes/shoulder_roll_r_link.STL" />
+        <mesh filename="package://tianyi2_urdf/meshes_convex/shoulder_roll_r_link.STL" />
       </geometry>
     </collision>
@@ -541,5 +541,5 @@
     <child link="shoulder_roll_r_link" />
     <axis xyz="1 0 0" />
-    <limit lower="-1.8325957145940461" upper="1.0471975511965976" effort="95.0" velocity="3.979350694547071" />
+    <limit lower="-2.6179938779914944" upper="0.2617993877991494" effort="95.0" velocity="3.979350694547071" />
   </joint>
   <link name="shoulder_yaw_r_link">
@@ -561,5 +561,5 @@
       <origin xyz="0 0 0" rpy="0 0 0" />
       <geometry>
-        <mesh filename="package://tianyi2_urdf/meshes/shoulder_yaw_r_link.STL" />
+        <mesh filename="package://tianyi2_urdf/meshes_convex/shoulder_yaw_r_link.STL" />
       </geometry>
     </collision>
@@ -590,5 +590,5 @@
       <origin xyz="0 0 0" rpy="0 0 0" />
       <geometry>
-        <mesh filename="package://tianyi2_urdf/meshes/elbow_pitch_r_link.STL" />
+        <mesh filename="package://tianyi2_urdf/meshes_convex/elbow_pitch_r_link.STL" />
       </geometry>
     </collision>
@@ -619,5 +619,5 @@
       <origin xyz="0 0 0" rpy="0 0 0" />
       <geometry>
-        <mesh filename="package://tianyi2_urdf/meshes/elbow_yaw_r_link.STL" />
+        <mesh filename="package://tianyi2_urdf/meshes_convex/elbow_yaw_r_link.STL" />
       </geometry>
     </collision>
@@ -648,5 +648,5 @@
       <origin xyz="0 0 0" rpy="0 0 0" />
       <geometry>
-        <mesh filename="package://tianyi2_urdf/meshes/wrist_pitch_r_link.STL" />
+        <mesh filename="package://tianyi2_urdf/meshes_convex/wrist_pitch_r_link.STL" />
       </geometry>
     </collision>
@@ -657,5 +657,5 @@
     <child link="wrist_pitch_r_link" />
     <axis xyz="0 1 0" />
-    <limit lower="-1.3089969389957472" upper="1.6580627893946132" effort="6.3" velocity="7.5398223686155035" />
+    <limit lower="-0.7853981633974483" upper="1.0471975511965976" effort="6.3" velocity="7.5398223686155035" />
   </joint>
   <link name="wrist_roll_r_link">
@@ -677,5 +677,5 @@
       <origin xyz="0 0 0" rpy="0 0 0" />
       <geometry>
-        <mesh filename="package://tianyi2_urdf/meshes/wrist_roll_r_link.STL" />
+        <mesh filename="package://tianyi2_urdf/meshes_convex/wrist_roll_r_link.STL" />
       </geometry>
     </collision>
@@ -686,5 +686,5 @@
     <child link="wrist_roll_r_link" />
     <axis xyz="1 0 0" />
-    <limit lower="-0.7853981633974483" upper="1.0471975511965976" effort="6.3" velocity="7.5398223686155035" />
+    <limit lower="-1.3089969389957472" upper="1.6580627893946132" effort="6.3" velocity="7.5398223686155035" />
   </joint>
   <link name="right_tcp_link">
@@ -706,5 +706,5 @@
       <origin xyz="0 0 0" rpy="0 0 0" />
       <geometry>
-        <mesh filename="package://tianyi2_urdf/meshes/right_tcp_link.STL" />
+        <mesh filename="package://tianyi2_urdf/meshes_convex/right_tcp_link.STL" />
       </geometry>
     </collision>
