Commit message: update

File: tianyi2_urdf/urdf/tianyi2.0_complete_with_hands.xacro (robot description, xacro)
@@ -16,5 +16,5 @@
       <collision>
         <origin xyz="0 0 0" rpy="0 0 0" />
-        <geometry><mesh filename="package://tianyi2_urdf/meshes/L_base_link.STL" /></geometry>
+        <geometry><mesh filename="package://tianyi2_urdf/meshes_convex/L_base_link.STL" /></geometry>
       </collision>
     </link>
@@ -33,5 +33,5 @@
       <collision>
         <origin xyz="0 0 0" rpy="0 0 0" />
-        <geometry><mesh filename="package://tianyi2_urdf/meshes/left_thumb_1.STL" /></geometry>
+        <geometry><mesh filename="package://tianyi2_urdf/meshes_convex/left_thumb_1.STL" /></geometry>
       </collision>
     </link>
@@ -57,5 +57,5 @@
       <collision>
         <origin xyz="0 0 0" rpy="0 0 0" />
-        <geometry><mesh filename="package://tianyi2_urdf/meshes/left_thumb_2.STL" /></geometry>
+        <geometry><mesh filename="package://tianyi2_urdf/meshes_convex/left_thumb_2.STL" /></geometry>
       </collision>
     </link>
@@ -81,5 +81,5 @@
       <collision>
         <origin xyz="0 0 0" rpy="0 0 0" />
-        <geometry><mesh filename="package://tianyi2_urdf/meshes/left_thumb_3.STL" /></geometry>
+        <geometry><mesh filename="package://tianyi2_urdf/meshes_convex/left_thumb_3.STL" /></geometry>
       </collision>
     </link>
@@ -106,5 +106,5 @@
       <collision>
         <origin xyz="0 0 0" rpy="0 0 0" />
-        <geometry><mesh filename="package://tianyi2_urdf/meshes/left_thumb_4.STL" /></geometry>
+        <geometry><mesh filename="package://tianyi2_urdf/meshes_convex/left_thumb_4.STL" /></geometry>
       </collision>
     </link>
@@ -131,5 +131,5 @@
       <collision>
         <origin xyz="0 0 0" rpy="0 0 0" />
-        <geometry><mesh filename="package://tianyi2_urdf/meshes/left_index_1.STL" /></geometry>
+        <geometry><mesh filename="package://tianyi2_urdf/meshes_convex/left_index_1.STL" /></geometry>
       </collision>
     </link>
@@ -155,5 +155,5 @@
       <collision>
         <origin xyz="0 0 0" rpy="0 0 0" />
-        <geometry><mesh filename="package://tianyi2_urdf/meshes/left_index_2.STL" /></geometry>
+        <geometry><mesh filename="package://tianyi2_urdf/meshes_convex/left_index_2.STL" /></geometry>
       </collision>
     </link>
@@ -180,5 +180,5 @@
       <collision>
         <origin xyz="0 0 0" rpy="0 0 0" />
-        <geometry><mesh filename="package://tianyi2_urdf/meshes/left_middle_1.STL" /></geometry>
+        <geometry><mesh filename="package://tianyi2_urdf/meshes_convex/left_middle_1.STL" /></geometry>
       </collision>
     </link>
@@ -204,5 +204,5 @@
       <collision>
         <origin xyz="0 0 0" rpy="0 0 0" />
-        <geometry><mesh filename="package://tianyi2_urdf/meshes/left_middle_2.STL" /></geometry>
+        <geometry><mesh filename="package://tianyi2_urdf/meshes_convex/left_middle_2.STL" /></geometry>
       </collision>
     </link>
@@ -229,5 +229,5 @@
       <collision>
         <origin xyz="0 0 0" rpy="0 0 0" />
-        <geometry><mesh filename="package://tianyi2_urdf/meshes/left_ring_1.STL" /></geometry>
+        <geometry><mesh filename="package://tianyi2_urdf/meshes_convex/left_ring_1.STL" /></geometry>
       </collision>
     </link>
@@ -253,5 +253,5 @@
       <collision>
         <origin xyz="0 0 0" rpy="0 0 0" />
-        <geometry><mesh filename="package://tianyi2_urdf/meshes/left_ring_2.STL" /></geometry>
+        <geometry><mesh filename="package://tianyi2_urdf/meshes_convex/left_ring_2.STL" /></geometry>
       </collision>
     </link>
@@ -278,5 +278,5 @@
       <collision>
         <origin xyz="0 0 0" rpy="0 0 0" />
-        <geometry><mesh filename="package://tianyi2_urdf/meshes/left_little_1.STL" /></geometry>
+        <geometry><mesh filename="package://tianyi2_urdf/meshes_convex/left_little_1.STL" /></geometry>
       </collision>
     </link>
@@ -302,5 +302,5 @@
       <collision>
         <origin xyz="0 0 0" rpy="0 0 0" />
-        <geometry><mesh filename="package://tianyi2_urdf/meshes/left_little_2.STL" /></geometry>
+        <geometry><mesh filename="package://tianyi2_urdf/meshes_convex/left_little_2.STL" /></geometry>
       </collision>
     </link>
@@ -335,5 +335,5 @@
       <collision>
         <origin xyz="0 0 0" rpy="0 0 0" />
-        <geometry><mesh filename="package://tianyi2_urdf/meshes/R_base_link.STL" /></geometry>
+        <geometry><mesh filename="package://tianyi2_urdf/meshes_convex/R_base_link.STL" /></geometry>
       </collision>
     </link>
@@ -352,5 +352,5 @@
       <collision>
         <origin xyz="0 0 0" rpy="0 0 0" />
-        <geometry><mesh filename="package://tianyi2_urdf/meshes/right_thumb_1.STL" /></geometry>
+        <geometry><mesh filename="package://tianyi2_urdf/meshes_convex/right_thumb_1.STL" /></geometry>
       </collision>
     </link>
@@ -376,5 +376,5 @@
       <collision>
         <origin xyz="0 0 0" rpy="0 0 0" />
-        <geometry><mesh filename="package://tianyi2_urdf/meshes/right_thumb_2.STL" /></geometry>
+        <geometry><mesh filename="package://tianyi2_urdf/meshes_convex/right_thumb_2.STL" /></geometry>
       </collision>
     </link>
@@ -399,5 +399,5 @@
       <collision>
         <origin xyz="0 0 0" rpy="0 0 0" />
-        <geometry><mesh filename="package://tianyi2_urdf/meshes/right_thumb_3.STL" /></geometry>
+        <geometry><mesh filename="package://tianyi2_urdf/meshes_convex/right_thumb_3.STL" /></geometry>
       </collision>
     </link>
@@ -424,5 +424,5 @@
       <collision>
         <origin xyz="0 0 0" rpy="0 0 0" />
-        <geometry><mesh filename="package://tianyi2_urdf/meshes/right_thumb_4.STL" /></geometry>
+        <geometry><mesh filename="package://tianyi2_urdf/meshes_convex/right_thumb_4.STL" /></geometry>
       </collision>
     </link>
@@ -449,5 +449,5 @@
       <collision>
         <origin xyz="0 0 0" rpy="0 0 0" />
-        <geometry><mesh filename="package://tianyi2_urdf/meshes/right_index_1.STL" /></geometry>
+        <geometry><mesh filename="package://tianyi2_urdf/meshes_convex/right_index_1.STL" /></geometry>
       </collision>
     </link>
@@ -473,5 +473,5 @@
       <collision>
         <origin xyz="0 0 0" rpy="0 0 0" />
-        <geometry><mesh filename="package://tianyi2_urdf/meshes/right_index_2.STL" /></geometry>
+        <geometry><mesh filename="package://tianyi2_urdf/meshes_convex/right_index_2.STL" /></geometry>
       </collision>
     </link>
@@ -498,5 +498,5 @@
       <collision>
         <origin xyz="0 0 0" rpy="0 0 0" />
-        <geometry><mesh filename="package://tianyi2_urdf/meshes/right_middle_1.STL" /></geometry>
+        <geometry><mesh filename="package://tianyi2_urdf/meshes_convex/right_middle_1.STL" /></geometry>
       </collision>
     </link>
@@ -522,5 +522,5 @@
       <collision>
         <origin xyz="0 0 0" rpy="0 0 0" />
-        <geometry><mesh filename="package://tianyi2_urdf/meshes/right_middle_2.STL" /></geometry>
+        <geometry><mesh filename="package://tianyi2_urdf/meshes_convex/right_middle_2.STL" /></geometry>
       </collision>
     </link>
@@ -547,5 +547,5 @@
       <collision>
         <origin xyz="0 0 0" rpy="0 0 0" />
-        <geometry><mesh filename="package://tianyi2_urdf/meshes/right_ring_1.STL" /></geometry>
+        <geometry><mesh filename="package://tianyi2_urdf/meshes_convex/right_ring_1.STL" /></geometry>
       </collision>
     </link>
@@ -571,5 +571,5 @@
       <collision>
         <origin xyz="0 0 0" rpy="0 0 0" />
-        <geometry><mesh filename="package://tianyi2_urdf/meshes/right_ring_2.STL" /></geometry>
+        <geometry><mesh filename="package://tianyi2_urdf/meshes_convex/right_ring_2.STL" /></geometry>
       </collision>
     </link>
@@ -596,5 +596,5 @@
       <collision>
         <origin xyz="0 0 0" rpy="0 0 0" />
-        <geometry><mesh filename="package://tianyi2_urdf/meshes/right_little_1.STL" /></geometry>
+        <geometry><mesh filename="package://tianyi2_urdf/meshes_convex/right_little_1.STL" /></geometry>
       </collision>
     </link>
@@ -620,5 +620,5 @@
       <collision>
         <origin xyz="0 0 0" rpy="0 0 0" />
-        <geometry><mesh filename="package://tianyi2_urdf/meshes/right_little_2.STL" /></geometry>
+        <geometry><mesh filename="package://tianyi2_urdf/meshes_convex/right_little_2.STL" /></geometry>
       </collision>
     </link>

File: tianyi2_urdf/urdf/tianyi2.0_urdf_with_hands.urdf (robot description, URDF)
Before this commit: robot tianyi2.0_complete, 51 links, 50 joints
Links:
- removed link body_yaw_link
- added link waist_yaw_link, mass 13.795395; collision mesh filename=package://tianyi2_urdf/meshes_convex/waist_yaw_link.STL; visual mesh filename=package://tianyi2_urdf/meshes/waist_yaw_link.STL
- link L_base_link: geometry collision mesh filename=package://tianyi2_urdf/meshes_convex/L_base_link.STL; visual mesh filename=package://tianyi2_urdf/meshes/L_base_link.STL
- link R_base_link: geometry collision mesh filename=package://tianyi2_urdf/meshes_convex/R_base_link.STL; visual mesh filename=package://tianyi2_urdf/meshes/R_base_link.STL
- link base: geometry collision mesh filename=package://tianyi2_urdf/meshes_convex/base.STL; visual mesh filename=package://tianyi2_urdf/meshes/base.STL
- link camera_head_link: geometry collision mesh filename=package://tianyi2_urdf/meshes_convex/camera_head_link.STL; visual mesh filename=package://tianyi2_urdf/meshes/camera_head_link.STL
- link elbow_pitch_l_link: geometry collision mesh filename=package://tianyi2_urdf/meshes_convex/elbow_pitch_l_link.STL; visual mesh filename=package://tianyi2_urdf/meshes/elbow_pitch_l_link.STL
- link elbow_pitch_r_link: geometry collision mesh filename=package://tianyi2_urdf/meshes_convex/elbow_pitch_r_link.STL; visual mesh filename=package://tianyi2_urdf/meshes/elbow_pitch_r_link.STL
- link elbow_yaw_l_link: geometry collision mesh filename=package://tianyi2_urdf/meshes_convex/elbow_yaw_l_link.STL; visual mesh filename=package://tianyi2_urdf/meshes/elbow_yaw_l_link.STL
- link elbow_yaw_r_link: geometry collision mesh filename=package://tianyi2_urdf/meshes_convex/elbow_yaw_r_link.STL; visual mesh filename=package://tianyi2_urdf/meshes/elbow_yaw_r_link.STL
- link first_leg_pitch_link: geometry collision mesh filename=package://tianyi2_urdf/meshes_convex/first_leg_pitch_link.S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; visual mesh filename=package://tianyi2_urdf/meshes/first_leg_pitch_link.STL
- link head_pitch_link: geometry collision mesh filename=package://tianyi2_urdf/meshes_convex/head_pitch_link.STL; visual mesh filename=package://tianyi2_urdf/meshes/head_pitch_link.STL
- link head_roll_link: geometry collision mesh filename=package://tianyi2_urdf/meshes_convex/head_roll_link.STL; visual mesh filename=package://tianyi2_urdf/meshes/head_roll_link.STL
- link head_yaw_link: geometry collision mesh filename=package://tianyi2_urdf/meshes_convex/head_yaw_link.STL; visual mesh filename=package://tianyi2_urdf/meshes/head_yaw_link.STL
- link left_index_1: geometry collision mesh filename=package://tianyi2_urdf/meshes_convex/left_index_1.STL; visual mesh filename=package://tianyi2_urdf/meshes/left_index_1.STL
- link left_index_2: geometry collision mesh filename=package://tianyi2_urdf/meshes_convex/left_index_2.STL; visual mesh filename=package://tianyi2_urdf/meshes/left_index_2.STL
- link left_little_1: geometry collision mesh filename=package://tianyi2_urdf/meshes_convex/left_little_1.STL; visual mesh filename=package://tianyi2_urdf/meshes/left_little_1.STL
- link left_little_2: geometry collision mesh filename=package://tianyi2_urdf/meshes_convex/left_little_2.STL; visual mesh filename=package://tianyi2_urdf/meshes/left_little_2.STL
- link left_middle_1: geometry collision mesh filename=package://tianyi2_urdf/meshes_convex/left_middle_1.STL; visual mesh filename=package://tianyi2_urdf/meshes/left_middle_1.STL
- link left_middle_2: geometry collision mesh filename=package://tianyi2_urdf/meshes_convex/left_middle_2.STL; visual mesh filename=package://tianyi2_urdf/meshes/left_middle_2.STL
- link left_ring_1: geometry collision mesh filename=package://tianyi2_urdf/meshes_convex/left_ring_1.STL; visual mesh filename=package://tianyi2_urdf/meshes/left_ring_1.STL
- link left_ring_2: geometry collision mesh filename=package://tianyi2_urdf/meshes_convex/left_ring_2.STL; visual mesh filename=package://tianyi2_urdf/meshes/left_ring_2.STL
- link left_tcp_link: geometry collision mesh filename=package://tianyi2_urdf/meshes_convex/left_tcp_link.STL; visual mesh filename=package://tianyi2_urdf/meshes/left_tcp_link.STL
- link left_thumb_1: geometry collision mesh filename=package://tianyi2_urdf/meshes_convex/left_thumb_1.STL; visual mesh filename=package://tianyi2_urdf/meshes/left_thumb_1.STL
- link left_thumb_2: geometry collision mesh filename=package://tianyi2_urdf/meshes_convex/left_thumb_2.STL; visual mesh filename=package://tianyi2_urdf/meshes/left_thumb_2.STL
- link left_thumb_3: geometry collision mesh filename=package://tianyi2_urdf/meshes_convex/left_thumb_3.STL; visual mesh filename=package://tianyi2_urdf/meshes/left_thumb_3.STL
- link left_thumb_4: geometry collision mesh filename=package://tianyi2_urdf/meshes_convex/left_thumb_4.STL; visual mesh filename=package://tianyi2_urdf/meshes/left_thumb_4.STL
- link right_index_1: geometry collision mesh filename=package://tianyi2_urdf/meshes_convex/right_index_1.STL; visual mesh filename=package://tianyi2_urdf/meshes/right_index_1.STL
- link right_index_2: geometry collision mesh filename=package://tianyi2_urdf/meshes_convex/right_index_2.STL; visual mesh filename=package://tianyi2_urdf/meshes/right_index_2.STL
- link right_little_1: geometry collision mesh filename=package://tianyi2_urdf/meshes_convex/right_little_1.STL; visual mesh filename=package://tianyi2_urdf/meshes/right_little_1.STL
- link right_little_2: geometry collision mesh filename=package://tianyi2_urdf/meshes_convex/right_little_2.STL; visual mesh filename=package://tianyi2_urdf/meshes/right_little_2.STL
- link right_middle_1: geometry collision mesh filename=package://tianyi2_urdf/meshes_convex/right_middle_1.STL; visual mesh filename=package://tianyi2_urdf/meshes/right_middle_1.STL
- link right_middle_2: geometry collision mesh filename=package://tianyi2_urdf/meshes_convex/right_middle_2.STL; visual mesh filename=package://tianyi2_urdf/meshes/right_middle_2.STL
- link right_ring_1: geometry collision mesh filename=package://tianyi2_urdf/meshes_convex/right_ring_1.STL; visual mesh filename=package://tianyi2_urdf/meshes/right_ring_1.STL
- link right_ring_2: geometry collision mesh filename=package://tianyi2_urdf/meshes_convex/right_ring_2.STL; visual mesh filename=package://tianyi2_urdf/meshes/right_ring_2.STL
- link right_tcp_link: geometry collision mesh filename=package://tianyi2_urdf/meshes_convex/right_tcp_link.STL; visual mesh filename=package://tianyi2_urdf/meshes/right_tcp_link.STL
- link right_thumb_1: geometry collision mesh filename=package://tianyi2_urdf/meshes_convex/right_thumb_1.STL; visual mesh filename=package://tianyi2_urdf/meshes/right_thumb_1.STL
- link right_thumb_2: geometry collision mesh filename=package://tianyi2_urdf/meshes_convex/right_thumb_2.STL; visual mesh filename=package://tianyi2_urdf/meshes/right_thumb_2.STL
- link right_thumb_3: geometry collision mesh filename=package://tianyi2_urdf/meshes_convex/right_thumb_3.STL; visual mesh filename=package://tianyi2_urdf/meshes/right_thumb_3.STL
- link right_thumb_4: geometry collision mesh filename=package://tianyi2_urdf/meshes_convex/right_thumb_4.STL; visual mesh filename=package://tianyi2_urdf/meshes/right_thumb_4.STL
- link second_leg_pitch_link: geometry collision mesh filename=package://tianyi2_urdf/meshes_convex/second_leg_pitch_link.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; visual mesh filename=package://tianyi2_urdf/meshes/second_leg_pitch_link.STL
- link shoulder_pitch_l_link: geometry collision mesh filename=package://tianyi2_urdf/meshes_convex/shoulder_pitch_l_link.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; visual mesh filename=package://tianyi2_urdf/meshes/shoulder_pitch_l_link.STL
- link shoulder_pitch_r_link: geometry collision mesh filename=package://tianyi2_urdf/meshes_convex/shoulder_pitch_r_link.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; visual mesh filename=package://tianyi2_urdf/meshes/shoulder_pitch_r_link.STL
- link shoulder_roll_l_link: geometry collision mesh filename=package://tianyi2_urdf/meshes_convex/shoulder_roll_l_link.S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; visual mesh filename=package://tianyi2_urdf/meshes/shoulder_roll_l_link.STL
- link shoulder_roll_r_link: geometry collision mesh filename=package://tianyi2_urdf/meshes_convex/shoulder_roll_r_link.S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; visual mesh filename=package://tianyi2_urdf/meshes/shoulder_roll_r_link.STL
- link shoulder_yaw_l_link: geometry collision mesh filename=package://tianyi2_urdf/meshes_convex/shoulder_yaw_l_link.STL; visual mesh filename=package://tianyi2_urdf/meshes/shoulder_yaw_l_link.STL
- link shoulder_yaw_r_link: geometry collision mesh filename=package://tianyi2_urdf/meshes_convex/shoulder_yaw_r_link.STL; visual mesh filename=package://tianyi2_urdf/meshes/shoulder_yaw_r_link.STL
- link waist_pitch_link: geometry collision mesh filename=package://tianyi2_urdf/meshes_convex/waist_pitch_link.STL; visual mesh filename=package://tianyi2_urdf/meshes/waist_pitch_link.STL
- link wrist_pitch_l_link: geometry collision mesh filename=package://tianyi2_urdf/meshes_convex/wrist_pitch_l_link.STL; visual mesh filename=package://tianyi2_urdf/meshes/wrist_pitch_l_link.STL
- link wrist_pitch_r_link: geometry collision mesh filename=package://tianyi2_urdf/meshes_convex/wrist_pitch_r_link.STL; visual mesh filename=package://tianyi2_urdf/meshes/wrist_pitch_r_link.STL
- link wrist_roll_l_link: geometry collision mesh filename=package://tianyi2_urdf/meshes_convex/wrist_roll_l_link.STL; visual mesh filename=package://tianyi2_urdf/meshes/wrist_roll_l_link.STL
- link wrist_roll_r_link: geometry collision mesh filename=package://tianyi2_urdf/meshes_convex/wrist_roll_r_link.STL; visual mesh filename=package://tianyi2_urdf/meshes/wrist_roll_r_link.STL
Joints:
- removed joint body_yaw_joint
- added joint waist_yaw_joint: type revolute, parent waist_pitch_link, child waist_yaw_link, origin xyz=0 0 0.07 rpy=0 0 0, axis 0 0 1, limit lower=-2.9670597283903604 upper=3.141592653589793 effort=143.0 velocity=4.71238898038469
- joint head_yaw_joint: parent body_yaw_link -> waist_yaw_link
- joint shoulder_pitch_l_joint: parent body_yaw_link -> waist_yaw_link
- joint shoulder_pitch_r_joint: parent body_yaw_link -> waist_yaw_link
- joint shoulder_roll_l_joint: limit lower=-1.0471975511965976 upper=1.8325957145940461 effort=95.0 velocity=3.979350694547071 -> lower=-0.2617993877991494 upper=2.6179938779914944 effort=95.0 velocity=3.979350694547071
- joint shoulder_roll_r_joint: limit lower=-1.8325957145940461 upper=1.0471975511965976 effort=95.0 velocity=3.979350694547071 -> lower=-2.6179938779914944 upper=0.2617993877991494 effort=95.0 velocity=3.979350694547071
- joint wrist_pitch_l_joint: limit lower=-1.3089969389957472 upper=1.6580627893946132 effort=6.3 velocity=7.5398223686155035 -> lower=-0.7853981633974483 upper=1.0471975511965976 effort=6.3 velocity=7.5398223686155035
- joint wrist_pitch_r_joint: limit lower=-1.3089969389957472 upper=1.6580627893946132 effort=6.3 velocity=7.5398223686155035 -> lower=-0.7853981633974483 upper=1.0471975511965976 effort=6.3 velocity=7.5398223686155035
- joint wrist_roll_l_joint: limit lower=-1.0471975511965976 upper=0.7853981633974483 effort=6.3 velocity=7.5398223686155035 -> lower=-1.6580627893946132 upper=1.3089969389957472 effort=6.3 velocity=7.5398223686155035
- joint wrist_roll_r_joint: limit lower=-0.7853981633974483 upper=1.0471975511965976 effort=6.3 velocity=7.5398223686155035 -> lower=-1.3089969389957472 upper=1.6580627893946132 effort=6.3 velocity=7.5398223686155035
